Commit message: 0717

File: urdf/ur5_peg.urdf (robot description, URDF)
Before this commit: robot universal_robot, 9 links, 8 joints
Links:
- link base_link: geometry collision mesh filename=meshes/ur5/collision/base.stl; visual mesh filename=./meshes/ur5/visual/base.obj
- link forearm_link: geometry collision mesh filename=./meshes/ur5/collision/forearm.stl; visual mesh filename=/meshes/ur5/visual/forearm.obj
- link peg: geometry collision mesh filename=./urdf/peg_hole_gazebo/peg/meshes/peg.STL; visual mesh filename=./urdf/peg_hole_gazebo/peg/meshes/peg.STL
- link shoulder_link: geometry collision mesh filename=./meshes/ur5/collision/shoulder.stl; visual mesh filename=/meshes/ur5/visual/shoulder.obj
- link upper_arm_link: geometry collision mesh filename=./meshes/ur5/collision/upperarm.stl; visual mesh filename=/meshes/ur5/visual/upperarm.obj
- link wrist_1_link: geometry collision mesh filename=./meshes/ur5/collision/wrist1.stl; visual mesh filename=./meshes/ur5/visual/wrist1.obj
- link wrist_2_link: geometry collision mesh filename=./meshes/ur5/collision/wrist2.stl; visual mesh filename=./meshes/ur5/visual/wrist2.obj
- link wrist_3_link: geometry collision mesh filename=./meshes/ur5/collision/wrist3.stl; visual mesh filename=./meshes/ur5/visual/wrist3.obj
