Commit message: 0814

File: urdf/peg_hole_gazebo/hole/urdf/new_hole1.urdf (robot description, URDF)
Before this commit: robot hole.SLDPRT, 1 links, 0 joints
Links:
- link hole: geometry collision mesh filename=../hole_stl/Hole_12.STL; visual mesh filename=../hole_stl/Hole_12.STL

File: urdf/peg_hole_gazebo/hole/urdf/new_hole2.urdf (robot description, URDF)
Before this commit: robot hole.SLDPRT, 1 links, 0 joints
Links:
- link hole: geometry collision mesh filename=../hole_stl/Hole_22.STL; visual mesh filename=../hole_stl/Hole_22.STL

File: urdf/peg_hole_gazebo/hole/urdf/new_hole3.urdf (robot description, URDF)
Before this commit: robot hole.SLDPRT, 1 links, 0 joints
Links:
- link hole: geometry collision mesh filename=../hole_stl/Hole_32.STL; visual mesh filename=../hole_stl/Hole_32.STL

File: urdf/peg_hole_gazebo/hole/urdf/new_hole4.urdf (robot description, URDF)
Before this commit: robot hole.SLDPRT, 1 links, 0 joints
Links:
- link hole: geometry collision mesh filename=../hole_stl/Hole_42.STL; visual mesh filename=../hole_stl/Hole_42.STL
